Commit message: Update to handle multi hands.

File: scripts/my_models/shadow/floating_shadow_multi.urdf (robot description, URDF)
Before this commit: robot shadowhand_motor, 32 links, 31 joints
Links:
- added link lh_arm_base, mass 10.0
- added link lh_arm_base_pitch, mass 0.01
- added link lh_arm_base_roll, mass 0.01
- added link lh_arm_base_x, mass 0.01
- added link lh_arm_base_y, mass 0.01
- added link lh_arm_base_z, mass 0.01
- added link lh_ffdistal, mass 0.012; collision mesh filename=package://sr_description/meshes/hand/F1.dae scale=0.001 0.001 0.001; visual mesh filename=package://sr_description/meshes/hand/F1.dae scale=0.001 0.001 0.001
- added link lh_ffknuckle, mass 0.008; collision cylinder length=0.014 radius=0.007; visual mesh filename=package://sr_description/meshes/hand/knuckle.dae scale=0.001 0.001 0.001
- added link lh_ffmiddle, mass 0.017; collision cylinder length=0.025 radius=0.007; collision sphere radius=0.007
- added link lh_ffproximal, mass 0.030; collision cylinder length=0.040 radius=0.007; visual mesh filename=package://sr_description/meshes/hand/F3.dae scale=0.001 0.001 0.001
- added link lh_fftip, mass 0.001
- added link lh_forearm, mass 1.8; collision box size=0.120 0.109 0.130; visual mesh filename=package://sr_description/meshes/hand/forearm_lite.dae scale=1.0 1.0 1.0
- added link lh_imu
- added link lh_manipulator
- added link lh_mfdistal, mass 0.012; collision mesh filename=package://sr_description/meshes/hand/F1.dae scale=0.001 0.001 0.001; visual mesh filename=package://sr_description/meshes/hand/F1.dae scale=0.001 0.001 0.001
- added link lh_mfknuckle, mass 0.008; collision cylinder length=0.014 radius=0.007; visual mesh filename=package://sr_description/meshes/hand/knuckle.dae scale=0.001 0.001 0.001
- added link lh_mfmiddle, mass 0.017; collision cylinder length=0.025 radius=0.007; collision sphere radius=0.007
- added link lh_mfproximal, mass 0.030; collision cylinder length=0.040 radius=0.007; visual mesh filename=package://sr_description/meshes/hand/F3.dae scale=0.001 0.001 0.001
- added link lh_mftip, mass 0.001
- added link lh_palm, mass 0.3; collision box size=0.018 0.024 0.004; collision box size=0.020 0.024 0.040
- added link lh_rfdistal, mass 0.012; collision mesh filename=package://sr_description/meshes/hand/F1.dae scale=0.001 0.001 0.001; visual mesh filename=package://sr_description/meshes/hand/F1.dae scale=0.001 0.001 0.001
- added link lh_rfknuckle, mass 0.008; collision cylinder length=0.014 radius=0.007; visual mesh filename=package://sr_description/meshes/hand/knuckle.dae scale=0.001 0.001 0.001
- added link lh_rfmiddle, mass 0.017; collision cylinder length=0.025 radius=0.007; collision sphere radius=0.007
- added link lh_rfproximal, mass 0.030; collision cylinder length=0.040 radius=0.007; visual mesh filename=package://sr_description/meshes/hand/F3.dae scale=0.001 0.001 0.001
- added link lh_rftip, mass 0.001
- added link lh_thbase, mass 0.010; collision sphere radius=0.011; visual box size=0.001 0.001 0.001
- added link lh_thdistal, mass 0.016; collision mesh filename=package://sr_description/meshes/hand/TH1_z.dae scale=0.001 0.001 0.001; visual mesh filename=package://sr_description/meshes/hand/TH1_z.dae scale=0.001 0.001 0.001
- added link lh_thhub, mass 0.005; collision sphere radius=0.010; visual box size=0.001 0.001 0.001
- added link lh_thmiddle, mass 0.020; collision cylinder length=0.018 radius=0.011; collision sphere radius=0.011
- added link lh_thproximal, mass 0.040; collision cylinder length=0.018 radius=0.012; visual mesh filename=package://sr_description/meshes/hand/TH3_z.dae scale=0.001 0.001 0.001
- added link lh_thtip, mass 0.001
Joints:
- added joint lh_FFJ1: type revolute, parent lh_ffmiddle, child lh_ffdistal, origin xyz=0 0 0.025 rpy=0 0 0, axis 1 0 0, limit lower=0 upper=1.57079632679 effort=2 velocity=2.0
- added joint lh_FFJ2: type revolute, parent lh_ffproximal, child lh_ffmiddle, origin xyz=0 0 0.045 rpy=0 0 0, axis 1 0 0, limit lower=0 upper=1.57079632679 effort=2 velocity=2.0
- added joint lh_FFJ3: type revolute, parent lh_ffknuckle, child lh_ffproximal, origin xyz=0 0 0 rpy=0 0 0, axis 1 0 0, limit lower=-0.261799387799 upper=1.57079632679 effort=2 velocity=2.0
- added joint lh_FFJ4: type revolute, parent lh_palm, child lh_ffknuckle, origin xyz=0.033 0 0.095 rpy=0 0 0, axis 0 -1.0 0, limit lower=-0.349065850399 upper=0.349065850399 effort=2 velocity=2.0
- added joint lh_FFtip: type fixed, parent lh_ffdistal, child lh_fftip, origin xyz=0 0 0.026 rpy=0 0 0
- added joint lh_MFJ1: type revolute, parent lh_mfmiddle, child lh_mfdistal, origin xyz=0 0 0.025 rpy=0 0 0, axis 1 0 0, limit lower=0 upper=1.57079632679 effort=2 velocity=2.0
- added joint lh_MFJ2: type revolute, parent lh_mfproximal, child lh_mfmiddle, origin xyz=0 0 0.045 rpy=0 0 0, axis 1 0 0, limit lower=0 upper=1.57079632679 effort=2 velocity=2.0
- added joint lh_MFJ3: type revolute, parent lh_mfknuckle, child lh_mfproximal, origin xyz=0 0 0 rpy=0 0 0, axis 1 0 0, limit lower=-0.261799387799 upper=1.57079632679 effort=2 velocity=2.0
- added joint lh_MFJ4: type revolute, parent lh_palm, child lh_mfknuckle, origin xyz=0.011 0 0.099 rpy=0 0 0, axis 0 -1.0 0, limit lower=-0.349065850399 upper=0.349065850399 effort=2 velocity=2.0
- added joint lh_MFtip: type fixed, parent lh_mfdistal, child lh_mftip, origin xyz=0 0 0.026 rpy=0 0 0
- added joint lh_RFJ1: type revolute, parent lh_rfmiddle, child lh_rfdistal, origin xyz=0 0 0.025 rpy=0 0 0, axis 1 0 0, limit lower=0 upper=1.57079632679 effort=2 velocity=2.0
- added joint lh_RFJ2: type revolute, parent lh_rfproximal, child lh_rfmiddle, origin xyz=0 0 0.045 rpy=0 0 0, axis 1 0 0, limit lower=0 upper=1.57079632679 effort=2 velocity=2.0
- added joint lh_RFJ3: type revolute, parent lh_rfknuckle, child lh_rfproximal, origin xyz=0 0 0 rpy=0 0 0, axis 1 0 0, limit lower=-0.261799387799 upper=1.57079632679 effort=2 velocity=2.0
- added joint lh_RFJ4: type revolute, parent lh_palm, child lh_rfknuckle, origin xyz=-0.011 0 0.095 rpy=0 0 0, axis 0 1.0 0, limit lower=-0.349065850399 upper=0.349065850399 effort=2 velocity=2.0
- added joint lh_RFtip: type fixed, parent lh_rfdistal, child lh_rftip, origin xyz=0 0 0.026 rpy=0 0 0
- added joint lh_THJ1: type revolute, parent lh_thmiddle, child lh_thdistal, origin xyz=0 0 0.032 rpy=0 0 -1.57079632679, axis 1 0 0, limit lower=-0.261799387799 upper=1.57079632679 effort=1.0 velocity=4.0
- added joint lh_THJ2: type revolute, parent lh_thhub, child lh_thmiddle, origin xyz=0 0 0 rpy=0 0 0, axis 0 -1 0, limit lower=-0.698131700798 upper=0.698131700798 effort=2.0 velocity=2.0
- added joint lh_THJ3: type fixed, parent lh_thproximal, child lh_thhub, origin xyz=0 0 0.038 rpy=0 0 0, axis 1 0 0
- added joint lh_THJ4: type revolute, parent lh_thbase, child lh_thproximal, origin xyz=0 0 0 rpy=0 0 0, axis 1.0 0 0, limit lower=0.0 upper=1.2217304764 effort=3 velocity=4.0
- added joint lh_THJ5: type revolute, parent lh_palm, child lh_thbase, origin xyz=0.034 -0.0085 0.029 rpy=0 0.785398163397 0.0, axis 0 0 -1.0, limit lower=-1.0471975512 upper=1.0471975512 effort=5.0 velocity=4.0
- added joint lh_Tx: type prismatic, parent world, child lh_arm_base_x, origin xyz=0 0 0 rpy=0 0 0, axis 1 0 0, limit lower=-500 upper=500 effort=87 velocity=2.1750
- added joint lh_Ty: type prismatic, parent lh_arm_base_x, child lh_arm_base_y, origin xyz=0 0 0 rpy=0 0 0, axis 0 1 0, limit lower=-500 upper=500 effort=87 velocity=2.1750
- added joint lh_Tz: type prismatic, parent lh_arm_base_y, child lh_arm_base_z, origin xyz=0 0 0 rpy=0 0 0, axis 0 0 1, limit lower=-500 upper=500 effort=87 velocity=2.1750
- added joint lh_WRJ1: type fixed, parent lh_forearm, child lh_palm, origin xyz=0 -0.015 0.149 rpy=-0.698131700798 0 0, axis 0 1.0 0
- added joint lh_arm_connector: type fixed, parent lh_arm_base, child lh_forearm, origin xyz=0.0 0.0 0.0 rpy=0 0 0 
- added joint lh_ee_fixed_joint: type fixed, parent lh_palm, child lh_manipulator, origin xyz=0.0 0.0 0.05 rpy=0.0 0.0 0.0
- added joint lh_palm_to_imu: type fixed, parent lh_palm, child lh_imu, origin xyz=0.01785 0.00765 0.049125 rpy=-1.5707963 3.141592 0.0
- added joint lh_pitch: type revolute, parent lh_arm_base_roll, child lh_arm_base_pitch, origin xyz=0 0 0 rpy=0 0 0, axis 0 1 0, limit lower=-500 upper=500 effort=87 velocity=2.1750
- added joint lh_roll: type revolute, parent lh_arm_base_z, child lh_arm_base_roll, origin xyz=0 0 0 rpy=0 0 0, axis 0 0 1, limit lower=-500 upper=500 effort=87 velocity=2.1750
- added joint lh_thtip: type fixed, parent lh_thdistal, child lh_thtip, origin xyz=0 0 0.0275 rpy=0 0 0
- added joint lh_yaw: type revolute, parent lh_arm_base_pitch, child lh_arm_base, origin xyz=0 0 0 rpy=0 0 0, axis 1 0 0, limit lower=-500 upper=500 effort=87 velocity=2.1750

Commit message: Update.

File: scripts/my_models/shadow/floating_shadow_multi.urdf (robot description, URDF)
Before this commit: robot shadowhand_motor, 63 links, 62 joints
Joints:
- joint lh_roll: axis 0 0 1 -> 1 0 0
- joint lh_yaw: axis 1 0 0 -> 0 0 1
